File: hw/ModuleInterface.kicad_pcb (KiCad board)
At the start: 2 copper layers, 38.1 x 99.1 mm, 41 parts, among them J1 clock_in, J2 gate_out_1, J3 gate_out_2, J4 gate_out_3, J5 gate_out_4, J7 Conn_02x09_Odd_Even, SW1 Rotary_Encoder, SW2 enter, SW3 func2, SW4 function

Commit message: minor mods
Parts:
- added J8: bus_R, Connector_PinHeader_2.54mm:PinHeader_1x10_P2.54mm_Vertical, F.Cu at (111.8, 119.4)
- added REF**: MountingHole_3.2mm_M3, MountingHole:MountingHole_3.2mm_M3, F.Cu at (80.0, 146.1)
- added REF**: MountingHole_3.2mm_M3, MountingHole:MountingHole_3.2mm_M3, F.Cu at (109.2, 61.0)
- C1, C2: footprint Capacitor_THT:C_Axial_L3.8mm_D2.6mm_P7.50mm_Horizontal -> Attenuverter:C_Axial_L4.8mm_D2.0mm_P2.54mm_Horizontal
- J7: value Conn_02x09_Odd_Even -> bus_L; footprint Connector_PinHeader_2.54mm:PinHeader_2x09_P2.54mm_Vertical -> Connector_PinHeader_2.54mm:PinHeader_1x10_P2.54mm_Vertical
- moved R5 22.6 mm to (78.7, 130.8)
- moved J7 22.5 mm to (78.7, 71.1)
- moved R2 22.2 mm to (100.3, 124.5), turned to 180 degrees
- moved C2 18.9 mm to (78.7, 128.3), turned to 90 degrees
- moved R1 14.5 mm to (100.3, 132.1), turned to 270 degrees
- moved R15 13.0 mm to (91.4, 73.7), turned to 90 degrees
- moved R17 13.0 mm to (91.4, 101.6), turned to 90 degrees
- moved R16 12.8 mm to (91.4, 87.6), turned to 90 degrees
- moved R18 12.8 mm to (91.4, 115.6), turned to 90 degrees
- moved C1 7.73 mm to (97.8, 129.5), turned to 90 degrees
- moved J1 1.27 mm to (85.1, 53.3)
- moved J2 1.27 mm to (85.1, 68.6), turned to 0 degrees
- moved J3 1.27 mm to (85.1, 82.5), turned to 0 degrees
- moved J4 1.27 mm to (85.1, 96.5), turned to 0 degrees
- moved J5 1.27 mm to (85.1, 110.5), turned to 0 degrees
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Connections:
- J7 pad 1: /Sheet62419879/clock_in -> +5V
- J7 pad 10: GND -> /Sheet62419879/select_3
- J7 pad 2: /Sheet62419879/seq_start -> /Sheet62419879/clock_in
- J7 pad 3: /Sheet62419879/gate_1 -> /Sheet62419879/seq_start
- J7 pad 4: /Sheet62419879/select_1 -> GND
- J7 pad 5: +5V -> /Sheet62419879/gate_1
- J7 pad 6: /Sheet62419879/gate_2 -> /Sheet62419879/select_1
- J7 pad 7: GND -> /Sheet62419879/gate_2
Routing:
- net /Sheet62419879/sw_func_2: track 48.5 -> 11.0 mm
- net /Sheet62419879/select_3: track 4.60 -> 35.1 mm
- net /Sheet62419879/sw_enter: track 49.2 -> 22.1 mm
- net /Sheet62419879/re_2: track 44.5 -> 17.4 mm
- net /Sheet62419879/select_2: track 4.34 -> 30.8 mm
- net /Sheet62419879/select_1: track 7.93 -> 33.4 mm
- net /Sheet62419879/sw_func_1: track 25.9 -> 6.88 mm
- net /Sheet62419879/seq_start: track 22.1 -> 40.4 mm
- net /Sheet62419879/gate_4: track 39.8 -> 27.2 mm
- net /Sheet62419879/re_1: track 31.7 -> 43.4 mm
- net +5V: track 107.4 -> 119.1 mm
- net /Sheet62419879/gate_3: track 30.8 -> 23.4 mm
- net /Sheet62419879/select_4: track 13.0 -> 18.5 mm
- net /Sheet62419879/clock_in: track 44.6 -> 39.8 mm
- net /Sheet62419879/gate_2: track 25.2 -> 20.6 mm
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Other:
- board text added: "button sequencer ver.2"
