File: hw/Panel.kicad_pcb (KiCad board)
At the start: 2 copper layers, 40.6 x 128.5 mm, 21 parts

Commit message: minor mods
Parts:
- removed Func: annotation_5.9mm_button, Attenuverter:annotation_5.9mm_button
- removed the fill/clear at (111.8, 110.5)
- added config/ratchet: MountingHole_5mm, MountingHole:MountingHole_5mm, F.Cu at (111.8, 127.0)
- added fill/clear: MountingHole_5mm, MountingHole:MountingHole_5mm, F.Cu at (111.8, 110.5)
