File: hw/_module_core.sch (KiCad schematic (older format))
At the start: 24 parts, among them J6 power_bus, J8 Conn_02x09_Odd_Even, Q1 2SC1815, SW5 SW_Push, U1 TL074, U2 ProMicro, U3 74HC595

Commit message: minor mods
Parts:
- removed J8: Conn_02x09_Odd_Even, Connector_PinHeader_2.54mm:PinHeader_2x09_P2.54mm_Vertical, symbol Connector_Generic:Conn_02x09_Odd_Even
- added C10, C8, C9: 0.1u, Attenuverter:C_Axial_L4.8mm_D2.0mm_P2.54mm_Horizontal, symbol Device:C
- added D11: 1N4148, Diode_THT:D_DO-35_SOD27_P2.54mm_Vertical_AnodeUp, symbol Diode:1N4148
- added D12, D13: D_Schottky, Diode_THT:D_DO-15_P2.54mm_Vertical_AnodeUp, symbol Device:D_Schottky
- added J10: bus_R, Connector_PinHeader_2.54mm:PinHeader_1x10_P2.54mm_Vertical, symbol Connector:Conn_01x10_Male
- added J9: bus_L, Connector_PinHeader_2.54mm:PinHeader_1x10_P2.54mm_Vertical, symbol Connector:Conn_01x10_Male
- added U4: L78L05_TO92, Package_TO_SOT_THT:TO-92_Inline_Wide, symbol Regulator_Linear:L78L05_TO92
- C5, C6, C7: footprint Capacitor_THT:C_Axial_L3.8mm_D2.6mm_P7.50mm_Horizontal -> Attenuverter:C_Axial_L4.8mm_D2.0mm_P2.54mm_Horizontal
- J6: footprint Connector_PinHeader_2.54mm:PinHeader_2x05_P2.54mm_Horizontal -> Connector_PinHeader_2.54mm:PinHeader_2x05_P2.54mm_Vertical
- Q1: footprint Package_TO_SOT_THT:TO-92_Inline -> Package_TO_SOT_THT:TO-92_Inline_Wide
Connections:
- net +12V: now also C8.2, D11.1 (K), D13.1 (K), U4.3 (VI); no longer J6.10 (Pin_10), J6.9 (Pin_9), U2.24 (RAW)
- net +5V: now also C9.2, D11.2 (A), J10.5 (Pin_5), J9.1 (Pin_1), U4.1 (VO)
- net -12V: now also C10.2, D12.2 (A); no longer C5.2, J6.1 (Pin_1), J6.2 (Pin_2)
- net GND: now also C5.2, C10.1, C8.1, C9.1, J10.1 (Pin_1), J10.10 (Pin_10), J9.4 (Pin_4), U4.2 (GND)
- net clock_in: now also J9.2 (Pin_2)
- net gate_1: now also J9.5 (Pin_5)
- net gate_2: now also J9.7 (Pin_7)
- net gate_3: now also J9.9 (Pin_9)
- net gate_4: now also J10.3 (Pin_3)
- net re_1: now also J10.7 (Pin_7)
- net re_2: now also J10.6 (Pin_6)
- net select_1: now also J9.6 (Pin_6)
- net select_2: now also J9.8 (Pin_8)
- net select_3: now also J9.10 (Pin_10)
- net select_4: now also J10.2 (Pin_2)
- net seq_start: now also J9.3 (Pin_3)
- net sw_enter: now also J10.9 (Pin_9)
- net sw_func_1: now also J10.4 (Pin_4)
- net sw_func_2: now also J10.8 (Pin_8)
- new net: D12.1 (K), J6.1 (Pin_1), J6.2 (Pin_2)
- new net: D13.2 (A), J6.10 (Pin_10), J6.9 (Pin_9)
- no-connect marks 9 -> 10
Other:
- moved on the sheet: C5, J6
